Commit message: naive_model

File: pkg/dobot_ws/src/dobot/description/dobot.urdf (robot description, URDF)
Before this commit: robot dobot, 4 links, 3 joints
Links:
- link base_link: geometry visual box size=0.16 0.16 0.056
- link link2: geometry visual cylinder length=0.08 radius=0.07
- link link3: geometry visual box size=0.07 0.04 0.14
- link link4: geometry visual box size=0.07 0.04 0.14
Joints:
- joint joint12: origin xyz=0 0 0.06 -> xyz=0 0 0.028 rpy=0 0 0
- joint joint23: origin xyz=0 0 0 -> xyz=0 0 0.08 rpy=0 0 0
- joint joint34: origin xyz=0 0.22 0.25 -> xyz=0 0 0.14 rpy=0 0 0

Commit message: urdf Xacro

File: pkg/dobot_ws/src/dobot/description/dobot.urdf (robot description, URDF)
Before this commit: robot dobot, 4 links, 3 joints
Links:
- added link link5; visual box size=0.09 0.05 0.07
Joints:
- added joint joint45: type continuous, parent link4, child link5, origin xyz=0 0 0.14 rpy=0 -${(joint23_degree+joint34_degree)/180*PI} 0
- joint joint12: origin xyz=0 0 0.028 rpy=0 0 0 -> xyz=0 0 0.028 rpy=0 0 ${joint12_degree/180*PI}
- joint joint23: origin xyz=0 0 0.08 rpy=0 0 0 -> xyz=0 0 0.08 rpy=0 ${joint23_degree/180*PI} 0
- joint joint34: origin xyz=0 0 0.14 rpy=0 0 0 -> xyz=0 0 0.14 rpy=0 ${joint34_degree/180*PI} 0
