Commit message: correct initial state

File: dobot/description/dobot.urdf (robot description, URDF)
Before this commit: robot dobot, 5 links, 4 joints
Joints:
- joint joint12: axis (none) -> 0 0 1
- joint joint23: axis (none) -> 0 1 0
- joint joint34: axis (none) -> 0 1 0
- joint joint45: axis (none) -> 0 1 0
